File: HARDWARE/KICAD/BUCK_CONVERTER_BOARD_V1.kicad_pcb (KiCad board)
At the start: 2 copper layers, 17.5 x 17.5 mm, 16 parts, among them J1 V/IN_CONN, J2 V/OUT_CONN, U1 LMR51430

Commit message: EDIT
CHANGED CURRENT RATING AND ADDED DIODE TO SCHEMATICS
Other:
- board text added: "~0.5-1A"
- board text removed: "(3A_PEAK)"
- board text removed: "2A_CONTINUOUS"
- board text removed: "5V_BUCK:"
Changed lines of the file:
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@@
-		)
-	)
-	(gr_text "(3A_PEAK)"
-		(at 105.5 81.774895 180)
-		(layer "B.SilkS")
-		(effects
-			(font
-				(size 0.8 0.8)
-				(thickness 0.1)
-			)
-			(justify left bottom mirror)
 		)
 	)
@@
 		)
 	)
-	(gr_text "5V_BUCK:"
-		(at 99.75 92.75 180)
+	(gr_text "~0.5-1A"
+		(at 107.034656 95.226176 0)
 		(layer "B.SilkS")
 		(effects
-			(font
-				(size 0.8 0.8)
-				(thickness 0.1)
-			)
-			(justify left bottom mirror)
-		)
-	)
-	(gr_text "2A_CONTINUOUS"
-		(at 108.75 95.25 0)
-		(layer "B.SilkS")
-		(effects
