File: HARDWARE/KICAD/BUCK_CONVERTER_BOARD_V1.kicad_sch (KiCad schematic)
At the start: 16 parts, among them J1 V/IN_CONN, J2 V/OUT_CONN, U1 LMR51430

Commit message: EDIT
CHANGED CURRENT RATING AND ADDED DIODE TO SCHEMATICS
Parts:
- added D1: D_Schottky, Diode_SMD:D_0402_1005Metric, symbol Device:D_Schottky
Connections:
- net GND: now also D1.2 (A)
- net SW: now also D1.1 (K)
Changed lines of the file:
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@@
 	(generator_version "9.0")
 	(paper "A4")
-	(text_box "LMR51430 Buck Converter 12V → 5V @ ~3A"
+	(text_box "LMR51430 Buck Converter 12V → 5V @ ~0.5A-1A"
 		(exclude_from_sim no)
 		(at 114.3 68.58 0)
@@
 	)
 	(junction
+		(at 160.02 115.57)
+		(diameter 0)
+		(color 0 0 0 0)
+	)
+	(junction
 		(at 140.97 115.57)
 		(diameter 0)
@@
 	)
 	(junction
+		(at 160.02 85.09)
+		(diameter 0)
+		(color 0 0 0 0)
+	)
+	(junction
 		(at 120.65 91.44)
 		(diameter 0)
@@
 	(wire
 		(pts
+			(xy 160.02 115.57) (xy 184.15 115.57)
+		)
+		(stroke
+			(width 0)
+			(type default)
+		)
+	)
+	(wire
+		(pts
+			(xy 160.02 85.09) (xy 158.75 85.09)
+		)
+		(stroke
+			(width 0)
+			(type default)
+		)
+	)
+	(wire
+		(pts
 			(xy 110.49 95.25) (xy 110.49 101.6)
 		)
@@
 	(wire
 		(pts
+			(xy 160.02 99.06) (xy 160.02 115.57)
+		)
+		(stroke
+			(width 0)
+			(type default)
+		)
+	)
+	(wire
+		(pts
+			(xy 160.02 85.09) (xy 160.02 91.44)
+		)
+		(stroke
+			(width 0)
+			(type default)
+		)
+	)
+	(wire
+		(pts
 			(xy 134.62 115.57) (xy 140.97 115.57)
 		)
@@
 	(wire
 		(pts
-			(xy 161.29 85.09) (xy 158.75 85.09)
+			(xy 161.29 85.09) (xy 160.02 85.09)
 		)
 		(stroke
@@
 	(wire
 		(pts
-			(xy 140.97 115.57) (xy 184.15 115.57)
+			(xy 140.97 115.57) (xy 160.02 115.57)
 		)
 		(stroke
@@
 					(unit 1)
 				)
+			)
+		)
+	)
+	(symbol
+		(lib_id "Device:D_Schottky")
+		(at 160.02 95.25 270)
+		(unit 1)
+		(exclude_from_sim no)
+		(in_bom yes)
+		(on_board yes)
+		(dnp no)
+		(fields_autoplaced yes)
+		(property "Reference" "D1"
+			(at 162.56 93.6624 90)
+			(effects
+				(font
+					(size 1.27 1.27)
+				)
+				(justify left)
+			)
+		)
+		(property "Value" "D_Schottky"
+			(at 162.56 96.2024 90)
+			(effects
+				(font
+					(size 1.27 1.27)
+				)
+				(justify left)
+			)
+		)
+		(property "Footprint" "Diode_SMD:D_0402_1005Metric"
+			(at 160.02 95.25 0)
+			(effects
+				(font
+					(size 1.27 1.27)
+				)
+				(hide yes)
+			)
+		)
+		(property "Datasheet" "~"
+			(at 160.02 95.25 0)
+			(effects
+				(font
+					(size 1.27 1.27)
+				)
+				(hide yes)
+			)
+		)
+		(property "Description" "Schottky diode"
+			(at 160.02 95.25 0)
+			(effects
+				(font
+					(size 1.27 1.27)
+				)
+				(hide yes)
+			)
+		)
+		(pin "1"
+		)
+		(pin "2"
+		)
+		(instances
+			(project ""
+				(path "/1fd95d44-98eb-480b-b5dd-6f6a0dbc39cb"
+					(reference "D1")
+					(unit 1)
+				)
